File: Platine/HM-LC-Sw1-FM.kicad_pcb (KiCad board)
At the start: 2 copper layers, 75 x 75 mm, 25 parts, among them J1 230V, J2 L_out, J3 S1, J4 S1, K1 FTR-LYCA024Y, Q1 BC546, SW1 CONFIG, U1 ArduinoProMini, U2 CC1101

Commit message: Images
Parts:
- Cp1: value Version 2.0.1 - 10/2019 -> Version 2.0.1 - 02/2020
Changed lines of the file:
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@@
   )
   (page A4)
+  (title_block
+    (title HM-LC-Sw1-FM)
+    (date 2020-02-01)
+    (rev V2.0.1)
+    (comment 1 "©S. Sternitzke")
+  )
   (layers
     (0 F.Cu signal)
@@
       (effects (font (size 1.2 1.2) (thickness 0.12)))
     )
-    (fp_text value "Version 2.0.1 - 10/2019" (at 0.762 2.032 90) (layer B.SilkS)
+    (fp_text value "Version 2.0.1 - 02/2020" (at 0.762 2.032 90) (layer B.SilkS)
       (effects (font (size 0.9 0.75) (thickness 0.12)) (justify mirror))
     )
